File: BreadboardPowerSupply_v2.sch (KiCad schematic (older format))
At the start: 15 parts

Commit message: Added 2nd text label.
Other:
- note added: "test 2"
Changed lines of the file:
@@
 Text Notes 3900 4700 0    50   ~ 0
 testing git\n
+Text Notes 4800 4650 0    50   ~ 0
+test 2
 $EndSCHEMATC
