File: BreadboardPowerSupply_v2.sch (KiCad schematic (older format))
At the start: 15 parts

Commit message: Added text label.
Other:
- note added: "testing git\n"
Changed lines of the file:
@@
 	1    0    0    -1
 $EndComp
+Text Notes 3900 4700 0    50   ~ 0
+testing git\n
 $EndSCHEMATC

Commit message: Test 3
Other:
- note added: "test 3"
- note added: "text sample 3"
Changed lines of the file:
@@
 Text Notes 3900 4700 0    50   ~ 0
 testing git\n
+Text Notes -313450 -185750 0    50   ~ 0
+text sample 3
+Text Notes 4750 4450 0    50   ~ 0
+test 3
 $EndSCHEMATC

Commit message: Removed experimental text.
Other:
- note removed: "test 3"
- note removed: "testing git\n"
Changed lines of the file:
@@
 	1    0    0    -1
 $EndComp
-Text Notes 3900 4700 0    50   ~ 0
-testing git\n
 Text Notes -313450 -185750 0    50   ~ 0
 text sample 3
-Text Notes 4750 4450 0    50   ~ 0
-test 3
 $EndSCHEMATC

Commit message: Components annotated.
Parts:
- gave numbers to parts that had none: 15
Changed lines of the file:
@@
 $EndDescr
 $Comp
-L Regulator_Linear:LM7805_TO220 U?
+L Regulator_Linear:LM7805_TO220 U1
 U 1 1 5B70E454
 P 5100 3300
-F 0 "U?" H 5100 3542 50  0000 C CNN
+F 0 "U1" H 5100 3542 50  0000 C CNN
 F 1 "LM7805_TO220" H 5100 3451 50  0000 C CNN
 F 2 "Package_TO_SOT_THT:TO-220-3_Vertical" H 5100 3525 50  0001 C CIN
@@
 $EndComp
 $Comp
-L Device:D D?
+L Device:D D1
 U 1 1 5B70E57A
 P 3550 3550
-F 0 "D?" V 3504 3629 50  0000 L CNN
+F 0 "D1" V 3504 3629 50  0000 L CNN
 F 1 "D" V 3595 3629 50  0000 L CNN
 F 2 "" H 3550 3550 50  0001 C CNN
@@
 $EndComp
 $Comp
-L Device:D D?
+L Device:D D2
 U 1 1 5B70E5E4
 P 3550 4050
-F 0 "D?" V 3504 4129 50  0000 L CNN
+F 0 "D2" V 3504 4129 50  0000 L CNN
 F 1 "D" V 3595 4129 50  0000 L CNN
 F 2 "" H 3550 4050 50  0001 C CNN
@@
 $EndComp
 $Comp
-L Device:D D?
+L Device:D D3
 U 1 1 5B70E602
 P 3900 3550
-F 0 "D?" V 3854 3629 50  0000 L CNN
+F 0 "D3" V 3854 3629 50  0000 L CNN
 F 1 "D" V 3945 3629 50  0000 L CNN
 F 2 "" H 3900 3550 50  0001 C CNN
@@
 $EndComp
 $Comp
-L Device:D D?
+L Device:D D4
 U 1 1 5B70E624
 P 3900 4050
-F 0 "D?" V 3854 4129 50  0000 L CNN
+F 0 "D4" V 3854 4129 50  0000 L CNN
 F 1 "D" V 3945 4129 50  0000 L CNN
 F 2 "" H 3900 4050 50  0001 C CNN
@@
 $EndComp
 $Comp
-L Device:CP1 C?
+L Device:CP1 C2
 U 1 1 5B70E6AA
 P 5550 3550
-F 0 "C?" H 5665 3596 50  0000 L CNN
+F 0 "C2" H 5665 3596 50  0000 L CNN
 F 1 "CP1" H 5665 3505 50  0000 L CNN
 F 2 "" H 5550 3550 50  0001 C CNN
@@
 $EndComp
 $Comp
-L Device:CP1 C?
+L Device:CP1 C1
 U 1 1 5B70E718
 P 4450 3550
-F 0 "C?" H 4565 3596 50  0000 L CNN
+F 0 "C1" H 4565 3596 50  0000 L CNN
 F 1 "CP1" H 4565 3505 50  0000 L CNN
 F 2 "" H 4450 3550 50  0001 C CNN
@@
 $EndComp
 $Comp
-L Device:LED D?
+L Device:LED D6
 U 1 1 5B70E7B0
 P 6900 4050
-F 0 "D?" V 6938 3933 50  0000 R CNN
+F 0 "D6" V 6938 3933 50  0000 R CNN
 F 1 "LED" V 6847 3933 50  0000 R CNN
 F 2 "" H 6900 4050 50  0001 C CNN
@@
 $EndComp
 $Comp
-L Device:LED D?
+L Device:LED D5
 U 1 1 5B70E80A
 P 5950 4050
-F 0 "D?" V 5988 3933 50  0000 R CNN
+F 0 "D5" V 5988 3933 50  0000 R CNN
 F 1 "LED" V 5897 3933 50  0000 R CNN
 F 2 "" H 5950 4050 50  0001 C CNN
@@
 $EndComp
 $Comp
-L Device:R R?
+L Device:R R1
 U 1 1 5B70E864
 P 5950 3550
-F 0 "R?" H 6020 3596 50  0000 L CNN
+F 0 "R1" H 6020 3596 50  0000 L CNN
 F 1 "R" H 6020 3505 50  0000 L CNN
 F 2 "" V 5880 3550 50  0001 C CNN
@@
 $EndComp
 $Comp
-L Device:R R?
+L Device:R R2
 U 1 1 5B70E8C2
 P 6900 3550
-F 0 "R?" H 6970 3596 50  0000 L CNN
+F 0 "R2" H 6970 3596 50  0000 L CNN
 F 1 "R" H 6970 3505 50  0000 L CNN
 F 2 "" V 6830 3550 50  0001 C CNN
@@
 $EndComp
 $Comp
-L Connector_Generic:Conn_02x02_Odd_Even J?
+L Connector_Generic:Conn_02x02_Odd_Even J3
 U 1 1 5B70E9B8
 P 7600 4100
-F 0 "J?" H 7650 4317 50  0000 C CNN
+F 0 "J3" H 7650 4317 50  0000 C CNN
 F 1 "Conn_02x02_Odd_Even" H 7650 4226 50  0000 C CNN
 F 2 "" H 7600 4100 50  0001 C CNN
@@
 $EndComp
 $Comp
-L Connector_Generic:Conn_02x02_Odd_Even J?
+L Connector_Generic:Conn_02x02_Odd_Even J2
 U 1 1 5B70EA3E
 P 7600 3300
-F 0 "J?" H 7650 3517 50  0000 C CNN
+F 0 "J2" H 7650 3517 50  0000 C CNN
 F 1 "Conn_02x02_Odd_Even" H 7650 3426 50  0000 C CNN
 F 2 "" H 7600 3300 50  0001 C CNN
@@
 $EndComp
 $Comp
-L Connector:Barrel_Jack_Switch J?
+L Connector:Barrel_Jack_Switch J1
 U 1 1 5B70ED22
 P 2950 3650
-F 0 "J?" H 3005 3967 50  0000 C CNN
+F 0 "J1" H 3005 3967 50  0000 C CNN
 F 1 "Barrel_Jack_Switch" H 3005 3876 50  0000 C CNN
 F 2 "" H 3000 3610 50  0001 C CNN
@@
 $EndComp
 $Comp
-L Switch:SW_DPDT_x2 SW?
+L Switch:SW_DPDT_x2 SW1
 U 1 1 5B70EDF7
 P 6450 3750
-F 0 "SW?" H 6450 4035 50  0000 C CNN
+F 0 "SW1" H 6450 4035 50  0000 C CNN
 F 1 "SW_DPDT_x2" H 6450 3944 50  0000 C CNN
 F 2 "" H 6450 3750 50  0001 C CNN

Commit message: Completed wiring, without nets.
Parts:
- C1: footprint (none) -> Capacitor_THT:CP_Radial_D10.0mm_P5.00mm_P7.50mm
- C2: footprint (none) -> Capacitor_THT:CP_Radial_D6.3mm_P2.50mm
- D1, D2, D3, D4: footprint (none) -> Diode_THT:D_DO-41_SOD81_P10.16mm_Horizontal
- D5, D6: footprint (none) -> LED_THT:LED_D5.0mm
- J1: footprint (none) -> Connector_BarrelJack:BarrelJack_CUI_PJ-102AH_Horizontal
- J2, J3: footprint (none) -> Connector_PinHeader_2.54mm:PinHeader_2x02_P2.54mm_Vertical
- R1, R2: footprint (none) -> Resistor_THT:R_Axial_DIN0207_L6.3mm_D2.5mm_P7.62mm_Horizontal
- SW1: footprint (none) -> digikey-footprints:Switch_Slide_11.6x4mm_EG1218
Connections:
- wire segments 0 -> 70
- no-connect marks 0 -> 2
Changed lines of the file:
@@
 F 0 "D1" V 3504 3629 50  0000 L CNN
 F 1 "D" V 3595 3629 50  0000 L CNN
-F 2 "" H 3550 3550 50  0001 C CNN
+F 2 "Diode_THT:D_DO-41_SOD81_P10.16mm_Horizontal" H 3550 3550 50  0001 C CNN
 F 3 "~" H 3550 3550 50  0001 C CNN
 	1    3550 3550
@@
 F 0 "D2" V 3504 4129 50  0000 L CNN
 F 1 "D" V 3595 4129 50  0000 L CNN
-F 2 "" H 3550 4050 50  0001 C CNN
+F 2 "Diode_THT:D_DO-41_SOD81_P10.16mm_Horizontal" H 3550 4050 50  0001 C CNN
 F 3 "~" H 3550 4050 50  0001 C CNN
 	1    3550 4050
@@
 F 0 "D3" V 3854 3629 50  0000 L CNN
 F 1 "D" V 3945 3629 50  0000 L CNN
-F 2 "" H 3900 3550 50  0001 C CNN
+F 2 "Diode_THT:D_DO-41_SOD81_P10.16mm_Horizontal" H 3900 3550 50  0001 C CNN
 F 3 "~" H 3900 3550 50  0001 C CNN
 	1    3900 3550
@@
 F 0 "D4" V 3854 4129 50  0000 L CNN
 F 1 "D" V 3945 4129 50  0000 L CNN
-F 2 "" H 3900 4050 50  0001 C CNN
+F 2 "Diode_THT:D_DO-41_SOD81_P10.16mm_Horizontal" H 3900 4050 50  0001 C CNN
 F 3 "~" H 3900 4050 50  0001 C CNN
 	1    3900 4050
@@
 F 0 "C2" H 5665 3596 50  0000 L CNN
 F 1 "CP1" H 5665 3505 50  0000 L CNN
-F 2 "" H 5550 3550 50  0001 C CNN
+F 2 "Capacitor_THT:CP_Radial_D6.3mm_P2.50mm" H 5550 3550 50  0001 C CNN
 F 3 "~" H 5550 3550 50  0001 C CNN
 	1    5550 3550
@@
 F 0 "C1" H 4565 3596 50  0000 L CNN
 F 1 "CP1" H 4565 3505 50  0000 L CNN
-F 2 "" H 4450 3550 50  0001 C CNN
+F 2 "Capacitor_THT:CP_Radial_D10.0mm_P5.00mm_P7.50mm" H 4450 3550 50  0001 C CNN
 F 3 "~" H 4450 3550 50  0001 C CNN
 	1    4450 3550
@@
 F 0 "D6" V 6938 3933 50  0000 R CNN
 F 1 "LED" V 6847 3933 50  0000 R CNN
-F 2 "" H 6900 4050 50  0001 C CNN
+F 2 "LED_THT:LED_D5.0mm" H 6900 4050 50  0001 C CNN
 F 3 "~" H 6900 4050 50  0001 C CNN
 	1    6900 4050
@@
 F 0 "D5" V 5988 3933 50  0000 R CNN
 F 1 "LED" V 5897 3933 50  0000 R CNN
-F 2 "" H 5950 4050 50  0001 C CNN
+F 2 "LED_THT:LED_D5.0mm" H 5950 4050 50  0001 C CNN
 F 3 "~" H 5950 4050 50  0001 C CNN
 	1    5950 4050
@@
 F 0 "R1" H 6020 3596 50  0000 L CNN
 F 1 "R" H 6020 3505 50  0000 L CNN
-F 2 "" V 5880 3550 50  0001 C CNN
+F 2 "Resistor_THT:R_Axial_DIN0207_L6.3mm_D2.5mm_P7.62mm_Horizontal" V 5880 3550 50  0001 C CNN
 F 3 "~" H 5950 3550 50  0001 C CNN
 	1    5950 3550
@@
 F 0 "R2" H 6970 3596 50  0000 L CNN
 F 1 "R" H 6970 3505 50  0000 L CNN
-F 2 "" V 6830 3550 50  0001 C CNN
+F 2 "Resistor_THT:R_Axial_DIN0207_L6.3mm_D2.5mm_P7.62mm_Horizontal" V 6830 3550 50  0001 C CNN
 F 3 "~" H 6900 3550 50  0001 C CNN
 	1    6900 3550
@@
 F 0 "J3" H 7650 4317 50  0000 C CNN
 F 1 "Conn_02x02_Odd_Even" H 7650 4226 50  0000 C CNN
-F 2 "" H 7600 4100 50  0001 C CNN
+F 2 "Connector_PinHeader_2.54mm:PinHeader_2x02_P2.54mm_Vertical" H 7600 4100 50  0001 C CNN
 F 3 "~" H 7600 4100 50  0001 C CNN
 	1    7600 4100
@@
 F 0 "J2" H 7650 3517 50  0000 C CNN
 F 1 "Conn_02x02_Odd_Even" H 7650 3426 50  0000 C CNN
-F 2 "" H 7600 3300 50  0001 C CNN
+F 2 "Connector_PinHeader_2.54mm:PinHeader_2x02_P2.54mm_Vertical" H 7600 3300 50  0001 C CNN
 F 3 "~" H 7600 3300 50  0001 C CNN
 	1    7600 3300
@@
 F 0 "J1" H 3005 3967 50  0000 C CNN
 F 1 "Barrel_Jack_Switch" H 3005 3876 50  0000 C CNN
-F 2 "" H 3000 3610 50  0001 C CNN
+F 2 "Connector_BarrelJack:BarrelJack_CUI_PJ-102AH_Horizontal" H 3000 3610 50  0001 C CNN
 F 3 "~" H 3000 3610 50  0001 C CNN
 	1    2950 3650
@@
 F 0 "SW1" H 6450 4035 50  0000 C CNN
 F 1 "SW_DPDT_x2" H 6450 3944 50  0000 C CNN
-F 2 "" H 6450 3750 50  0001 C CNN
+F 2 "digikey-footprints:Switch_Slide_11.6x4mm_EG1218" H 6450 3750 50  0001 C CNN
 F 3 "" H 6450 3750 50  0001 C CNN
 	1    6450 3750
@@
 Text Notes -313450 -185750 0    50   ~ 0
 text sample 3
+Wire Wire Line
+	3550 3700 3550 3750
+Wire Wire Line
+	3900 3700 3900 3850
+Wire Wire Line
+	3550 4200 3550 4450
+Wire Wire Line
+	3550 4450 3750 4450
+Wire Wire Line
+	3900 4450 3900 4200
+Wire Wire Line
+	3900 3400 3900 3200
+Wire Wire Line
+	3900 3200 3750 3200
+Wire Wire Line
+	3550 3200 3550 3400
+Wire Wire Line
+	3250 3550 3400 3550
+Wire Wire Line
+	3400 3550 3400 3750
+Wire Wire Line
+	3400 3750 3550 3750
+Connection ~ 3550 3750
+Wire Wire Line
+	3550 3750 3550 3900
+Wire Wire Line
+	3250 3750 3250 3850
+Wire Wire Line
+	3250 3850 3900 3850
+Connection ~ 3900 3850
+Wire Wire Line
+	3900 3850 3900 3900
+NoConn ~ 3250 3650
+Wire Wire Line
+	3750 3200 3750 3100
+Wire Wire Line
+	3750 3100 4450 3100
+Wire Wire Line
+	4450 3100 4450 3300
+Connection ~ 3750 3200
+Wire Wire Line
+	3750 3200 3550 3200
+Wire Wire Line
+	4800 3300 4450 3300
+Connection ~ 4450 3300
+Wire Wire Line
+	4450 3300 4450 3400
+Wire Wire Line
+	3750 4450 3750 4550
+Wire Wire Line
+	3750 4550 4450 4550
+Wire Wire Line
+	4450 4550 4450 3700
+Connection ~ 3750 4450
+Wire Wire Line
+	3750 4450 3900 4450
+Wire Wire Line
+	4450 4550 5100 4550
+Wire Wire Line
+	5550 4550 5550 3700
+Connection ~ 4450 4550
+Wire Wire Line
+	5100 3600 5100 4550
+Connection ~ 5100 4550
+Wire Wire Line
+	5100 4550 5550 4550
+Wire Wire Line
+	5400 3300 5550 3300
+Wire Wire Line
+	5550 3300 5550 3400
+Wire Wire Line
+	5550 3300 5950 3300
+Wire Wire Line
+	5950 3300 5950 3400
+Connection ~ 5550 3300
+Wire Wire Line
+	5950 3700 5950 3900
+Wire Wire Line
+	5550 4550 5950 4550
+Wire Wire Line
+	5950 4550 5950 4200
+Connection ~ 5550 4550
+Wire Wire Line
+	5950 3300 6200 3300
+Wire Wire Line
+	6200 3300 6200 3750
+Wire Wire Line
+	6200 3750 6250 3750
+Connection ~ 5950 3300
+Wire Wire Line
+	5950 4550 6900 4550
+Wire Wire Line
+	6900 4550 6900 4200
+Connection ~ 5950 4550
+Wire Wire Line
+	6900 3900 6900 3700
+Wire Wire Line
+	6650 3650 6650 3300
+Wire Wire Line
+	6650 3300 6900 3300
+Wire Wire Line
+	6900 3300 6900 3400
+Wire Wire Line
+	6900 3300 7250 3300
+Connection ~ 6900 3300
+Wire Wire Line
+	7250 3300 7250 3800
+Wire Wire Line
+	7250 4100 7400 4100
+Connection ~ 7250 3300
+Wire Wire Line
+	7250 3300 7400 3300
+Wire Wire Line
+	6900 4550 7250 4550
+Wire Wire Line
+	7250 4550 7250 4200
+Wire Wire Line
+	7250 4200 7350 4200
+Connection ~ 6900 4550
+Wire Wire Line
+	7350 4200 7350 3650
+Wire Wire Line
+	7350 3400 7400 3400
+Connection ~ 7350 4200
+Wire Wire Line
+	7350 4200 7400 4200
+Wire Wire Line
+	7900 3300 8050 3300
+Wire Wire Line
+	8050 3300 8050 3050
+Wire Wire Line
+	8050 3050 7250 3050
+Wire Wire Line
+	7250 3050 7250 3300
+Wire Wire Line
+	7900 3400 8050 3400
+Wire Wire Line
+	8050 3400 8050 3650
+Wire Wire Line
+	8050 3650 7350 3650
+Connection ~ 7350 3650
+Wire Wire Line
+	7350 3650 7350 3400
+Wire Wire Line
+	7900 4100 8050 4100
+Wire Wire Line
+	8050 4100 8050 3800
+Wire Wire Line
+	8050 3800 7250 3800
+Connection ~ 7250 3800
+Wire Wire Line
+	7250 3800 7250 4100
+Wire Wire Line
+	7900 4200 8050 4200
+Wire Wire Line
+	8050 4200 8050 4550
+Wire Wire Line
+	8050 4550 7250 4550
+Connection ~ 7250 4550
+NoConn ~ 6650 3850
 $EndSCHEMATC

Commit message: Added power flags.
Changed lines of the file:
@@
 L Switch:SW_DPDT_x2 SW1
 U 1 1 5B70EDF7
-P 6450 3750
-F 0 "SW1" H 6450 4035 50  0000 C CNN
-F 1 "SW_DPDT_x2" H 6450 3944 50  0000 C CNN
-F 2 "digikey-footprints:Switch_Slide_11.6x4mm_EG1218" H 6450 3750 50  0001 C CNN
-F 3 "" H 6450 3750 50  0001 C CNN
-	1    6450 3750
+P 6450 3300
+F 0 "SW1" H 6450 3585 50  0000 C CNN
+F 1 "SW_DPDT_x2" H 6450 3494 50  0000 C CNN
+F 2 "digikey-footprints:Switch_Slide_11.6x4mm_EG1218" H 6450 3300 50  0001 C CNN
+F 3 "" H 6450 3300 50  0001 C CNN
+	1    6450 3300
 	1    0    0    -1
 $EndComp
@@
 	3750 3200 3750 3100
 Wire Wire Line
-	3750 3100 4450 3100
+	3750 3100 4100 3100
 Wire Wire Line
 	4450 3100 4450 3300
@@
 	3750 4450 3900 4450
 Wire Wire Line
-	4450 4550 5100 4550
+	4450 4550 4800 4550
 Wire Wire Line
 	5550 4550 5550 3700
@@
 	5950 4550 5950 4200
 Connection ~ 5550 4550
-Wire Wire Line
-	5950 3300 6200 3300
-Wire Wire Line
-	6200 3300 6200 3750
-Wire Wire Line
-	6200 3750 6250 3750
 Connection ~ 5950 3300
 Wire Wire Line
@@
 	6900 3900 6900 3700
 Wire Wire Line
-	6650 3650 6650 3300
+	6650 3200 6650 3300
 Wire Wire Line
 	6650 3300 6900 3300
@@
 	8050 4550 7250 4550
 Connection ~ 7250 4550
-NoConn ~ 6650 3850
+NoConn ~ 6650 3400
+Wire Wire Line
+	5950 3300 6250 3300
+$Comp
+L power:PWR_FLAG #FLG0101
+U 1 1 5B72F9CB
+P 4100 3100
+F 0 "#FLG0101" H 4100 3175 50  0001 C CNN
+F 1 "PWR_FLAG" H 4100 3274 50  0000 C CNN
+F 2 "" H 4100 3100 50  0001 C CNN
+F 3 "~" H 4100 3100 50  0001 C CNN
+	1    4100 3100
+	1    0    0    -1
+$EndComp
+Connection ~ 4100 3100
+Wire Wire Line
+	4100 3100 4450 3100
+$Comp
+L power:PWR_FLAG #FLG0102
+U 1 1 5B72FA0C
+P 4800 4550
+F 0 "#FLG0102" H 4800 4625 50  0001 C CNN
+F 1 "PWR_FLAG" H 4800 4724 50  0000 C CNN
+F 2 "" H 4800 4550 50  0001 C CNN
+F 3 "~" H 4800 4550 50  0001 C CNN
+	1    4800 4550
+	1    0    0    -1
+$EndComp
+Connection ~ 4800 4550
+Wire Wire Line
+	4800 4550 5100 4550
 $EndSCHEMATC

Commit message: Added net labels.
Connections:
- net labels added: 5V, V+, V-
Changed lines of the file:
@@
 Wire Wire Line
 	4800 4550 5100 4550
+Text Label 6150 4550 0    50   ~ 0
+V-
+Text Label 4200 3100 0    50   ~ 0
+V+
+Text Label 5650 3300 0    50   ~ 0
+5V
 $EndSCHEMATC

Commit message: Completed ERC.
Connections:
- net labels added: Vin, Vout
- net labels removed: 5V, V+
Changed lines of the file:
@@
 V-
 Text Label 4200 3100 0    50   ~ 0
-V+
+Vin
 Text Label 5650 3300 0    50   ~ 0
-5V
+Vout
 $EndSCHEMATC
