File: BreadboardPowerSupply_v2.sch (KiCad schematic (older format))
At the start: 15 parts, among them J1 Barrel_Jack_Switch, J2 Conn_02x02_Odd_Even, J3 Conn_02x02_Odd_Even, SW1 SW_DPDT_x2, U1 LM7805_TO220

Commit message: Added descriptibe text, and finished with the schematic.
Other:
- note added: "Bridge rectifier"
- note added: "On/Off \nswitch"
- note added: "Output\npower\nindicator"
- note added: "Power input"
- note added: "Power output"
- note added: "Power\nindicator"
- note added: "Voltage regulator"
Changed lines of the file:
@@
 Wire Notes Line
 	8100 2800 7100 2800
+Text Notes 2600 2800 0    50   ~ 0
+Power input
+Text Notes 3500 2800 0    50   ~ 0
+Bridge rectifier
+Text Notes 4350 2800 0    50   ~ 0
+Voltage regulator
+Text Notes 5750 2800 0    50   ~ 0
+Power\nindicator
+Text Notes 6200 2800 0    50   ~ 0
+On/Off \nswitch
+Text Notes 6750 2800 0    50   ~ 0
+Output\npower\nindicator
+Text Notes 7100 2800 0    50   ~ 0
+Power output
 $EndSCHEMATC

Commit message: Placement of footprints almost done. Fixed an incorrect association for C1.
Parts:
- C1: footprint Capacitor_THT:CP_Radial_D10.0mm_P5.00mm_P7.50mm -> Capacitor_THT:CP_Radial_D10.0mm_P5.00mm
Changed lines of the file:
@@
 F 0 "C1" H 4565 3596 50  0000 L CNN
 F 1 "CP1" H 4565 3505 50  0000 L CNN
-F 2 "Capacitor_THT:CP_Radial_D10.0mm_P5.00mm_P7.50mm" H 4450 3550 50  0001 C CNN
+F 2 "Capacitor_THT:CP_Radial_D10.0mm_P5.00mm" H 4450 3550 50  0001 C CNN
 F 3 "~" H 4450 3550 50  0001 C CNN
 	1    4450 3550

Commit message: Added additional net names for power.
Connections:
- net labels added: V1, V2, Vout1, Vout2
- net labels removed: Vout
Changed lines of the file:
@@
 Vin
 Text Label 5650 3300 0    50   ~ 0
-Vout
+Vout1
 Wire Notes Line
 	3450 2800 3450 4650
@@
 Text Notes 7100 2800 0    50   ~ 0
 Power output
+Text Label 3300 3550 0    50   ~ 0
+V1
+Text Label 3300 3850 0    50   ~ 0
+V2
+Text Label 6800 3300 0    50   ~ 0
+Vout2
 $EndSCHEMATC

Commit message: Replaced capacitor symbols as per IEC 60617 and IEEE 315, Clause 2.2.1 Style 1.
Parts:
- removed C1: CP1, Capacitor_THT:CP_Radial_D10.0mm_P5.00mm, symbol Device:CP1
- removed C2: CP1, Capacitor_THT:CP_Radial_D6.3mm_P2.50mm, symbol Device:CP1
- added C?: CP, Capacitor_THT:CP_Radial_D10.0mm_P5.00mm, symbol Device:CP
- added C?: CP, Capacitor_THT:CP_Radial_D6.3mm_P2.50mm, symbol Device:CP
Changed lines of the file:
@@
 EESchema Schematic File Version 4
+LIBS:BreadboardPowerSupply_v2-cache
 EELAYER 26 0
 EELAYER END
@@
 	1    3900 4050
 	0    1    1    0
-$EndComp
-$Comp
-L Device:CP1 C2
-U 1 1 5B70E6AA
-P 5550 3550
-F 0 "C2" H 5665 3596 50  0000 L CNN
-F 1 "CP1" H 5665 3505 50  0000 L CNN
-F 2 "Capacitor_THT:CP_Radial_D6.3mm_P2.50mm" H 5550 3550 50  0001 C CNN
-F 3 "~" H 5550 3550 50  0001 C CNN
-	1    5550 3550
-	1    0    0    -1
-$EndComp
-$Comp
-L Device:CP1 C1
-U 1 1 5B70E718
-P 4450 3550
-F 0 "C1" H 4565 3596 50  0000 L CNN
-F 1 "CP1" H 4565 3505 50  0000 L CNN
-F 2 "Capacitor_THT:CP_Radial_D10.0mm_P5.00mm" H 4450 3550 50  0001 C CNN
-F 3 "~" H 4450 3550 50  0001 C CNN
-	1    4450 3550
-	1    0    0    -1
 $EndComp
 $Comp
@@
 Text Label 6800 3300 0    50   ~ 0
 Vout2
+$Comp
+L Device:CP C?
+U 1 1 5B9F5330
+P 4450 3550
+F 0 "C?" H 4568 3596 50  0000 L CNN
+F 1 "CP" H 4568 3505 50  0000 L CNN
+F 2 "Capacitor_THT:CP_Radial_D10.0mm_P5.00mm" H 4488 3400 50  0001 C CNN
+F 3 "~" H 4450 3550 50  0001 C CNN
+	1    4450 3550
+	1    0    0    -1
+$EndComp
+$Comp
+L Device:CP C?
+U 1 1 5B9F55AF
+P 5550 3550
+F 0 "C?" H 5668 3596 50  0000 L CNN
+F 1 "CP" H 5668 3505 50  0000 L CNN
+F 2 "Capacitor_THT:CP_Radial_D6.3mm_P2.50mm" H 5588 3400 50  0001 C CNN
+F 3 "~" H 5550 3550 50  0001 C CNN
+	1    5550 3550
+	1    0    0    -1
+$EndComp
 $EndSCHEMATC

Commit message: Replaced designation of LEDs with DS as per  IEEE 315, Clause 22.4
Parts:
- gave numbers to parts that had none: 2
- renumbered D5 to DS5, D6 to DS6
Changed lines of the file:
@@
 $EndComp
 $Comp
-L Device:LED D6
+L Device:LED DS6
 U 1 1 5B70E7B0
 P 6900 4050
-F 0 "D6" V 6938 3933 50  0000 R CNN
+F 0 "DS6" V 6938 3933 50  0000 R CNN
 F 1 "LED" V 6847 3933 50  0000 R CNN
 F 2 "LED_THT:LED_D5.0mm" H 6900 4050 50  0001 C CNN
@@
 $EndComp
 $Comp
-L Device:LED D5
+L Device:LED DS5
 U 1 1 5B70E80A
 P 5950 4050
-F 0 "D5" V 5988 3933 50  0000 R CNN
+F 0 "DS5" V 5988 3933 50  0000 R CNN
 F 1 "LED" V 5897 3933 50  0000 R CNN
 F 2 "LED_THT:LED_D5.0mm" H 5950 4050 50  0001 C CNN
@@
 Vout2
 $Comp
-L Device:CP C?
+L Device:CP C1
 U 1 1 5B9F5330
 P 4450 3550
-F 0 "C?" H 4568 3596 50  0000 L CNN
+F 0 "C1" H 4568 3596 50  0000 L CNN
 F 1 "CP" H 4568 3505 50  0000 L CNN
 F 2 "Capacitor_THT:CP_Radial_D10.0mm_P5.00mm" H 4488 3400 50  0001 C CNN
@@
 $EndComp
 $Comp
-L Device:CP C?
+L Device:CP C2
 U 1 1 5B9F55AF
 P 5550 3550
-F 0 "C?" H 5668 3596 50  0000 L CNN
+F 0 "C2" H 5668 3596 50  0000 L CNN
 F 1 "CP" H 5668 3505 50  0000 L CNN
 F 2 "Capacitor_THT:CP_Radial_D6.3mm_P2.50mm" H 5588 3400 50  0001 C CNN

Commit message: Added  non-class letter N for fenced-in areas.
Other:
- note added: "N1 - Power input"
- note added: "N2 - Bridge rectifier"
- note added: "N3 - Voltage regulator"
- note added: "N4 -\nPower\nindicator"
- note added: "N5 - \nOn/Off \nswitch"
- note added: "N6 -\nOutput\npower\nindicator"
- note added: "N7 - Power output"
- note removed: "Bridge rectifier"
- note removed: "On/Off \nswitch"
- note removed: "Output\npower\nindicator"
- note removed: "Power input"
- note removed: "Power output"
- note removed: "Power\nindicator"
- note removed: "Voltage regulator"
Changed lines of the file:
@@
 	4350 4650 5700 4650
-Wire Notes Line
-	5700 4650 5700 2800
 Wire Notes Line
 	5700 2800 4350 2800
 Wire Notes Line
-	5750 2800 5750 4650
-Wire Notes Line
 	5750 4650 6150 4650
 Wire Notes Line
-	6150 4650 6150 2800
-Wire Notes Line
 	6150 2800 5750 2800
-Wire Notes Line
-	6200 2800 6200 4650
 Wire Notes Line
 	6200 4650 6700 4650
@@
 	6750 4650 7050 4650
 Wire Notes Line
-	7050 4650 7050 2800
-Wire Notes Line
 	7050 2800 6750 2800
-Wire Notes Line
-	7100 2800 7100 4650
 Wire Notes Line
 	7100 4650 8100 4650
@@
 Wire Notes Line
 	8100 2800 7100 2800
-Text Notes 2600 2800 0    50   ~ 0
-Power input
-Text Notes 3500 2800 0    50   ~ 0
-Bridge rectifier
-Text Notes 4350 2800 0    50   ~ 0
-Voltage regulator
-Text Notes 5750 2800 0    50   ~ 0
-Power\nindicator
-Text Notes 6200 2800 0    50   ~ 0
-On/Off \nswitch
-Text Notes 6750 2800 0    50   ~ 0
-Output\npower\nindicator
-Text Notes 7100 2800 0    50   ~ 0
-Power output
 Text Label 3300 3550 0    50   ~ 0
 V1
@@
 	1    0    0    -1
 $EndComp
+Wire Notes Line
+	5700 4650 5700 2800
+Wire Notes Line
+	5750 2800 5750 4650
+Wire Notes Line
+	7100 2800 7100 4650
+Wire Notes Line
+	7050 4650 7050 2800
+Wire Notes Line
+	6200 2800 6200 4650
+Wire Notes Line
+	6150 4650 6150 2800
+Text Notes 7100 2800 0    50   ~ 0
+N7 - Power output
+Text Notes 6750 2800 0    50   ~ 0
+N6 -\nOutput\npower\nindicator
+Text Notes 6200 2800 0    50   ~ 0
+N5 - \nOn/Off \nswitch
+Text Notes 5750 2800 0    50   ~ 0
+N4 -\nPower\nindicator
+Text Notes 4350 2800 0    50   ~ 0
+N3 - Voltage regulator
+Text Notes 3500 2800 0    50   ~ 0
+N2 - Bridge rectifier
+Text Notes 2600 2800 0    50   ~ 0
+N1 - Power input
 $EndSCHEMATC
